File: logic.brd (EAGLE design)
At the start: 37.8 x 80 mm, 86 parts, among them CON11 PINHEAD_1X03-2, CON12 PINHEAD_1X03-2, CON2 PINHEAD_2X02-PTH-2-MALE, CON3 PINHEAD_2X04-PLS-2, CON4 CON-3P-TABS, CON5 PINHEAD_2X02-PTH-2-MALE, CON6 PINHEAD_2X02-PTH-2-MALE, CON7 PINHEAD_2X02-PTH-2-MALE, IC1 STM32F105RCT6, IC10 LM75-TSSOP8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

Commit message: blah
Parts:
- moved C11 23.0 mm to (-6.15, 18.4)
- moved C29 23.0 mm to (-6.15, 16.9)
- moved L4 0.71 mm to (0.00, 45.0)
- moved L3 0.58 mm to (0.00, 52.0)
- moved L1 0.41 mm to (0.00, 27.0)
- moved R23 0.20 mm to (5.45, 75.0)
- moved R24 0.20 mm to (6.55, 75.0)
- moved R25 0.20 mm to (7.65, 75.0)
