File: logic.sch (EAGLE design)
At the start: 86 parts, among them CON11 PINHEAD_1X03-2, CON12 PINHEAD_1X03-2, CON2 PINHEAD_2X02-PTH-2-MALE, CON3 PINHEAD_2X04-PLS-2, CON4 CON-3P-TABS, CON5 PINHEAD_2X02-PTH-2-MALE, CON6 PINHEAD_2X02-PTH-2-MALE, CON7 PINHEAD_2X02-PTH-2-MALE, IC1 STM32F105RCT6, IC10 LM75-TSSOP8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

Commit message: blah
Other:
- moved on the sheet: C11, C13, C22, C25, C28, C29, C30, CON2, CON3, CON5, CON6, CON7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
